File: tc36k/pcb/gamma-omega-tc36k-routed.kicad_pcb (KiCad board)
At the start: 2 copper layers, 232.8 x 111.4 mm, 45 parts

Commit message: Update text to TC36K v1.1.0, move traces by centre hole, shorten traces
Add reset label, restore ground plane
Parts:
- moved S20 0.44 mm to (262.9, 83.1)
- moved S17 0.44 mm to (104.5, 130.2)
- moved H5 0.44 mm to (131.6, 54.4)
- moved S13 0.44 mm to (118.5, 114.2)
- moved H6 0.44 mm to (180.9, 54.4)
- moved S9 0.44 mm to (99.2, 57.8)
- moved S3 0.44 mm to (49.6, 66.1)
- moved _1 0.44 mm to (156.2, 76.0)
- moved S18 0.44 mm to (119.1, 144.4)
- moved S7 0.44 mm to (88.7, 90.2)
- moved S27 0.44 mm to (213.3, 57.8)
- moved S28 0.44 mm to (209.1, 103.7)
- moved S15 0.44 mm to (131.2, 82.7)
- moved S4 0.44 mm to (68.9, 92.1)
- moved S23 0.44 mm to (240.6, 75.4)
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Routing:
- net R12: track 297.3 -> 216.2 mm
- net R2: track 363.1 -> 296.5 mm
- net R10: track 367.1 -> 310.5 mm
- net R13: track 381.6 -> 333.9 mm
- net C2: track 231.2 -> 195.9 mm
- net R9: track 241.8 -> 209.2 mm
- net R6: track 215.7 -> 184.6 mm
- net R1: track 263.3 -> 235.5 mm
- net R4: track 251.5 -> 225.5 mm
- net R11: track 215.6 -> 190.8 mm
- net C12: track 231.2 -> 210.6 mm
- net R8: track 224.1 -> 212.0 mm
- net C7: track 124.9 -> 114.4 mm
- net R7: track 253.9 -> 244.2 mm
- net C1: track 209.2 -> 199.9 mm
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- added copper zone on B.Cu, net GND
- added copper zone on F.Cu, net GND
Other:
- outline, holes or cut-outs redrawn
- board text added: "Diode-free using Graph Theory"
- board text added: "Ergogen v4.1.0 & KiCad v9.0.4"
- board text added: "Gamma Omega 'TC36K' v1.1.0"
- board text added: "Original design Tokyo June 2025"
- board text added: "Reset"
- board text removed: "Designed Tokyo June 2025, with Ergogen v4.1.0 & KiCad v9.0.2"
